File: keyball-row-staggered/right-top-1/keyball-row-staggered-right.kicad_pcb (KiCad board)
At the start: 2 copper layers, 178.2 x 113.8 mm, 14 parts

Commit message: 発注ファイル作成
Parts:
- removed the REF** at (67.8, 124.5)
- removed the REF** at (729.2, 540.8)
- removed the REF** at (62.3, 134.2)
- removed the REF** at (50.8, 128.9)
Other:
- board size 178.2 x 113.8 mm -> 152.4 x 95.3 mm
